File: raspberrypi_zerow_uhat/raspberrypi_zerow_uhat.kicad_pcb (KiCad board)
At the start: 2 copper layers, 65 x 30 mm, 5 parts, among them J1 GPIO_CONNECTOR

Commit message: work-in-progress
Other:
- net class Default removed
