File: uhat_spdif_transmitter/uhat_spdif_transmitter/uhat_spdif_transmitter.kicad_pcb (KiCad board)
At the start: 4 copper layers, 65 x 30 mm, 76 parts, among them J1 GPIO_CONNECTOR, J2 Conn_02x03_Odd_Even, J3 Conn_01x03_Pin, J4 Conn_02x03_Odd_Even, SW1 TS24CA, U1 PLR237/T10BK, U10 USBLC6-2SC6, U2 LR8103A-T12, U4 W25Q32JVSSIQ, U5 24LC256T-I/SN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

Commit message: Change Optical Connector + other stuff
Connections:
- C12 pad 1: Net-(U1-VCC) -> Net-(U1-GND)
- C13 pad 1: Net-(U6-VCC) -> Net-(U6-GND)
- FB1 pad 2: Net-(U1-VCC) -> Net-(U1-GND)
- FB2 pad 2: Net-(U6-VCC) -> Net-(U6-GND)
- U1 pad 1: Net-(U1-VCC) -> /OPT1
- U1 pad 2: GND -> Net-(U1-GND)
- U1 pad 3: /OPT1 -> GND
- U6 pad 1: Net-(U6-VCC) -> /OPT2
- U6 pad 2: GND -> Net-(U6-GND)
- U6 pad 3: /OPT2 -> GND
Routing:
- net Net-(U6-GND): track 0.00 -> 6.86 mm
- net Net-(U6-VCC): track 5.33 -> 0.00 mm
- net /OPT2: track 51.9 -> 46.8 mm
- net Net-(U1-GND): track 0.00 -> 4.98 mm
- net Net-(U1-VCC): track 4.49 -> 0.00 mm
- net /OPT1: track 37.0 -> 33.2 mm
- net Net-(U4-IO3): track 2.67 -> 1.71 mm, vias 1 -> 0
Changed lines of the file:
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@@
 	(net 2 "+5V")
 	(net 3 "+1V2")
-	(net 4 "Net-(U1-VCC)")
+	(net 4 "Net-(U1-GND)")
 	(net 5 "GND")
 	(net 6 "/GPIO4_GPIO_GCLK")
-	(net 7 "Net-(U6-VCC)")
+	(net 7 "Net-(U6-GND)")
 	(net 8 "Net-(D1-K)")
 	(net 9 "/GPIO17_GEN0")
@@
 			(layers "*.Cu" "*.Mask")
 			(remove_unused_layers no)
-			(net 7 "Net-(U6-VCC)")
-			(pinfunction "VCC")
+			(net 59 "/OPT2")
+			(pinfunction "VOUT")
 			(pintype "unspecified")
 		)
@@
 			(layers "*.Cu" "*.Mask")
 			(remove_unused_layers no)
-			(net 5 "GND")
-			(pinfunction "GND")
+			(net 7 "Net-(U6-GND)")
+			(pinfunction "VCC")
 			(pintype "unspecified")
 		)
@@
 			(layers "*.Cu" "*.Mask")
 			(remove_unused_layers no)
-			(net 59 "/OPT2")
-			(pinfunction "VOUT")
+			(net 5 "GND")
+			(pinfunction "GND")
 			(pintype "unspecified")
 		)
@@
 			(layers "F.Cu" "F.Mask" "F.Paste")
 			(roundrect_rratio 0.25)
-			(net 7 "Net-(U6-VCC)")
+			(net 7 "Net-(U6-GND)")
 			(pintype "passive")
 		)
@@
 			(layers "*.Cu" "*.Mask")
 			(remove_unused_layers no)
-			(net 4 "Net-(U1-VCC)")
-			(pinfunction "VCC")
+			(net 57 "/OPT1")
+			(pinfunction "VOUT")
 			(pintype "unspecified")
 		)
@@
 			(layers "*.Cu" "*.Mask")
 			(remove_unused_layers no)
-			(net 5 "GND")
-			(pinfunction "GND")
+			(net 4 "Net-(U1-GND)")
+			(pinfunction "VCC")
 			(pintype "unspecified")
 		)
@@
 			(layers "*.Cu" "*.Mask")
 			(remove_unused_layers no)
-			(net 57 "/OPT1")
-			(pinfunction "VOUT")
+			(net 5 "GND")
+			(pinfunction "GND")
 			(pintype "unspecified")
 		)
@@
 			(layers "F.Cu" "F.Mask" "F.Paste")
 			(roundrect_rratio 0.25)
-			(net 7 "Net-(U6-VCC)")
+			(net 7 "Net-(U6-GND)")
 			(pintype "passive")
 		)
@@
 			(layers "F.Cu" "F.Mask" "F.Paste")
 			(roundrect_rratio 0.25)
-			(net 4 "Net-(U1-VCC)")
+			(net 4 "Net-(U1-GND)")
 			(pintype "passive")
 		)
@@
 			(layers "F.Cu" "F.Mask" "F.Paste")
 			(roundrect_rratio 0.25)
-			(net 4 "Net-(U1-VCC)")
+			(net 4 "Net-(U1-GND)")
 			(pintype "passive")
 		)
@@
 	)
 	(segment
-		(start 152.517 112.233)
-		(end 152.492 112.258)
-		(width 0.2)
+		(start 153.802 111.028)
+		(end 155.032 112.258)
+		(width 0.25)
 		(layer "F.Cu")
 		(net 4)
 	)
 	(segment
-		(start 153.802 109.068)
-		(end 152.517 109.068)
-		(width 0.2)
+		(start 152.517 109.068)
+		(end 153.802 109.068)
+		(width 0.25)
 		(layer "F.Cu")
 		(net 4)
 	)
 	(segment
-		(start 152.517 109.068)
-		(end 152.517 112.233)
-		(width 0.2)
+		(start 153.802 109.068)
+		(end 153.802 111.028)
+		(width 0.25)
 		(layer "F.Cu")
 		(net 4)
@@
 	(segment
 		(start 165.052 108.568)
-		(end 165.052 111.318)
+		(end 165.052 109.588)
+		(width 0.2)
+		(layer "F.Cu")
+		(net 7)
+	)
+	(segment
+		(start 165.052 109.588)
+		(end 167.722 112.258)
 		(width 0.2)
 		(layer "F.Cu")
@@
 	)
 	(segment
-		(start 165.052 111.318)
-		(end 165.992 112.258)
+		(start 167.722 112.258)
+		(end 168.532 112.258)
 		(width 0.2)
 		(layer "F.Cu")
@@
 	)
 	(segment
-		(start 141.167 116.673)
-		(end 141.167 116.433)
-		(width 0.2)
-		(layer "F.Cu")
-		(net 51)
-	)
-	(segment
-		(start 140.657 117.183)
-		(end 141.167 116.673)
-		(width 0.2)
-		(layer "F.Cu")
-		(net 51)
-	)
-	(segment
 		(start 140.522 117.048)
 		(end 140.657 117.183)
@@
 		(net 51)
 	)
-	(via
-		(at 141.167 116.433)
-		(size 0.4)
-		(drill 0.3)
-		(layers "F.Cu" "B.Cu")
-		(net 51)
-	)
 	(segment
 		(start 126.3795 111.568)
@@
 	)
 	(segment
+		(start 152.517 112.233)
+		(end 152.492 112.258)
+		(width 0.2)
+		(layer "F.Cu")
+		(net 57)
+	)
+	(segment
 		(start 130.032 110.9155)
 		(end 130.032 111.818)
@@
 	)
 	(segment
+		(start 150.782 116.068)
+		(end 149.782 117.068)
+		(width 0.2)
+		(layer "B.Cu")
+		(net 57)
+	)
+	(segment
 		(start 135.032 120.068)
 		(end 145.532 120.068)
@@
 	)
 	(segment
+		(start 148.532 117.068)
+		(end 149.782 117.068)
+		(width 0.2)
+		(layer "B.Cu")
+		(net 57)
+	)
+	(segment
 		(start 130.032 115.068)
 		(end 135.032 120.068)
@@
 	)
 	(segment
-		(start 152.762 117.068)
-		(end 157.572 112.258)
+		(start 150.782 113.968)
+		(end 150.782 116.068)
 		(width 0.2)
 		(layer "B.Cu")
@@
 	)
 	(segment
-		(start 148.532 117.068)
-		(end 152.762 117.068)
+		(start 152.492 112.258)
+		(end 150.782 113.968)
 		(width 0.2)
 		(layer "B.Cu")
@@
 	(segment
 		(start 148.282 118.318)
-		(end 165.012 118.318)
+		(end 159.282 118.318)
 		(width 0.2)
 		(layer "B.Cu")
@@
 	)
 	(segment
-		(start 129.032 111.818)
-		(end 129.032 115.068)
+		(start 165.992 112.258)
+		(end 159.932 118.318)
+		(width 0.2)
+		(layer "B.Cu")
+		(net 59)
+	)
+	(segment
+		(start 159.932 118.318)
+		(end 159.282 118.318)
 		(width 0.2)
 		(layer "B.Cu")
@@
 	)
 	(segment
-		(start 165.012 118.318)
-		(end 171.072 112.258)
+		(start 129.032 111.818)
+		(end 129.032 115.068)
 		(width 0.2)
 		(layer "B.Cu")
